Commit message: Tennis ball urdf and ranfom motion generator ready

File: xarm6_control_trainig/urdf/tennis_robot_alone.urdf.xacro (robot description, xacro)
@@ -1,4 +1,4 @@
 <?xml version="1.0"?>
-<robot name="tennis_ball">
+<robot xmlns:xacro="http://www.ros.org/wiki/xacro"  name="tennis_ball">
   <!-- Material Definition -->
   <material name="yellow">
@@ -122,6 +122,6 @@
       <child link="x_link"/>
       <axis xyz="1 0 0"/>
-      <limit effort="100" velocity="0.1" lower="-0.3" upper="0.3"/>
-      <dynamics damping="10.0" friction="10.0"/>
+      <limit effort="50" velocity="0.01" lower="-0.3" upper="0.3"/>
+      <dynamics damping="100.0" friction="100.0"/>
   </joint>
   <joint name="y_joint" type="prismatic">
@@ -130,6 +130,6 @@
       <child link="y_link"/>
       <axis xyz="0 1 0"/>
-      <limit effort="100" velocity="0.1" lower="-0.3" upper="0.3"/>
-      <dynamics damping="10.0" friction="10.0"/>
+      <limit effort="50" velocity="0.01" lower="-0.3" upper="0.3"/>
+      <dynamics damping="100.0" friction="100.0"/>
   </joint>
   <joint name="z_joint" type="prismatic">
@@ -138,6 +138,6 @@
       <child link="z_link"/>
       <axis xyz="0 0 1"/>
-      <limit effort="100" velocity="0.1" lower="-0.3" upper="0.3"/>
-      <dynamics damping="10.0" friction="10.0"/>
+      <limit effort="50" velocity="0.01" lower="-0.3" upper="0.3"/>
+      <dynamics damping="100.0" friction="100.0"/>
   </joint>
   <joint name="fixed_joint" type="fixed">
@@ -146,33 +146,5 @@
       <child link="ball"/>
   </joint>
-  <gazebo reference="base_link">
-    <material>Gazebo/Black</material>
-  </gazebo>
-  <gazebo reference="x_link">
-    <material>Gazebo/Black</material>
-  </gazebo>
-  <gazebo reference="y_link">
-    <material>Gazebo/Black</material>
-  </gazebo>
-  <gazebo reference="z_link">
-    <material>Gazebo/Black</material>
-  </gazebo>
-  <gazebo reference="ball">
-    <material>Gazebo/Yellow</material>
-  </gazebo>
-  <gazebo>
-      <plugin name="gazebo_ros_joint_state_publisher"
-          filename="libgazebo_ros_joint_state_publisher.so">
-          <update_rate>20</update_rate>
-          <joint_name>x_joint</joint_name>
-          <joint_name>y_joint</joint_name>
-          <joint_name>z_joint</joint_name>
-      </plugin>
-  </gazebo>
-  <gazebo>
-      <plugin name="gazebo_ros_joint_pose_trajectory"
-          filename="libgazebo_ros_joint_pose_trajectory.so">
-          <update_rate>2</update_rate>
-      </plugin>
-  </gazebo>
+  <xacro:include filename="gazebo_plugin.xacro" />
 </robot>
+<!-- ros2 topic pub -1 /set_joint_trajectory trajectory_msgs/msg/JointTrajectory  '{header: {frame_id: world}, joint_names: [x_joint, y_joint, z_joint], points: [{positions: {0.3,0.3,0.3}, velocities: {0.02,0.01,0.01}}}]} -->
