Commit message: Adding velocity control

File: xarm6_control_trainig/urdf/gazebo_plugin.xacro (robot description, xacro)
@@ -28,5 +28,5 @@
       <plugin name="gazebo_ros_joint_pose_trajectory"
           filename="libgazebo_ros_joint_pose_trajectory.so">
-          <update_rate>20</update_rate>
+          <update_rate>30</update_rate>
       </plugin>
   </gazebo>
@@ -40,5 +40,5 @@
   <gazebo>
       <plugin name="gazebo_ros_control" filename="libgazebo_ros_control.so">
-      <update_rate>20</update_rate>
+      <update_rate>30</update_rate>
     </plugin>
   </gazebo>

File: xarm6_control_trainig/urdf/tennis_robot_alone.urdf.xacro (robot description, xacro)
@@ -14,5 +14,5 @@
     <visual>
       <geometry>
-        <box size="0.6 0.01 0.01"/>
+        <box size="1.2 0.01 0.01"/>
       </geometry>
       <material name="black"/>
@@ -20,5 +20,5 @@
     <collision>
       <geometry>
-        <box size="0.6 0.01 0.01"/>
+        <box size="1.2 0.01 0.01"/>
       </geometry>
     </collision>
@@ -26,5 +26,5 @@
       <mass value="10"/>
       <origin rpy="0 0 0" xyz="0 0 0"/>
-      <inertia ixx="0.008333333333" ixy="0" ixz="0" iyy="0.1541666667" iyz="0" izz="0.1541666667"/>
+      <inertia ixx="0.008333333333" ixy="0" ixz="0" iyy="0.0.06041666667" iyz="0" izz="0.0.06041666667"/>
     </inertial>
   </link>
@@ -34,5 +34,5 @@
       <origin xyz="0 0 0" rpy="0 0 0"/>
       <geometry>
-        <box size="0.01 0.6 0.01"/>
+        <box size="0.01 1.2 0.01"/>
       </geometry>
       <material name="black"/>
@@ -41,5 +41,5 @@
       <origin xyz="0 0 0" rpy="0 0 0"/>
       <geometry>
-        <box size="0.01 0.6 0.01"/>
+        <box size="0.01 1.2 0.01"/>
       </geometry>
     </collision>
@@ -47,5 +47,5 @@
       <mass value="0.5"/>
       <origin rpy="0 0 0" xyz="0 0 0"/>
-      <inertia ixx="0.01541666667" ixy="0" ixz="0" iyy="0.0008333333333" iyz="0" izz="0.01541666667"/>
+      <inertia ixx="0.0.06041666667" ixy="0" ixz="0" iyy="0.0008333333333" iyz="0" izz="0.0.06041666667"/>
     </inertial>
   </link>
@@ -54,5 +54,5 @@
       <origin xyz="0 0 0" rpy="0 0 0"/>
       <geometry>
-        <box size="0.01 0.01 0.6"/>
+        <box size="0.01 0.01 1.2"/>
       </geometry>
       <material name="black"/>
@@ -61,5 +61,5 @@
       <origin xyz="0 0 0" rpy="0 0 0"/>
       <geometry>
-        <box size="0.01 0.01 0.6"/>
+        <box size="0.01 0.01 1.2"/>
       </geometry>
     </collision>
@@ -67,5 +67,5 @@
       <mass value="0.5"/>
       <origin rpy="0 0 0" xyz="0 0 0"/>
-      <inertia ixx="0.01541666667" ixy="0" ixz="0" iyy="0.01541666667" iyz="0" izz="0.0008333333333"/>
+      <inertia ixx="0.0.06041666667" ixy="0" ixz="0" iyy="0.0.06041666667" iyz="0" izz="0.0008333333333"/>
     </inertial>
   </link>
@@ -118,17 +118,17 @@
   </joint>
   <joint name="x_joint" type="prismatic">
-      <origin xyz="0 0.305 0" rpy="0 0 0"/>
+      <origin xyz="0 0.605 0" rpy="0 0 0"/>
       <parent link="base_link"/>
       <child link="x_link"/>
       <axis xyz="1 0 0"/>
-      <limit effort="50" velocity="0.01" lower="-0.3" upper="0.3"/>
+      <limit effort="50" velocity="0.01" lower="-0.6" upper="0.6"/>
       <dynamics damping="100.0" friction="100.0"/>
   </joint>
   <joint name="y_joint" type="prismatic">
-      <origin xyz="0 0 0.305" rpy="0 0 0"/>
+      <origin xyz="0 0 0.605" rpy="0 0 0"/>
       <parent link="x_link"/>
       <child link="y_link"/>
       <axis xyz="0 1 0"/>
-      <limit effort="50" velocity="0.01" lower="-0.3" upper="0.3"/>
+      <limit effort="50" velocity="0.01" lower="-0.6" upper="0.6"/>
       <dynamics damping="100.0" friction="100.0"/>
   </joint>
@@ -138,5 +138,5 @@
       <child link="z_link"/>
       <axis xyz="0 0 1"/>
-      <limit effort="50" velocity="0.01" lower="-0.3" upper="0.3"/>
+      <limit effort="50" velocity="0.01" lower="-0.6" upper="0.6"/>
       <dynamics damping="100.0" friction="100.0"/>
   </joint>
