Commit message: cylindrical tennis mover and velocity controller

File: xarm6_control_trainig/urdf/tennis_robot.urdf.xacro (robot description, xacro)
@@ -1,4 +1,5 @@
 <?xml version="1.0"?>
 <robot xmlns:xacro="http://www.ros.org/wiki/xacro"  name="tennis_ball">
+  <!-- <xacro:include filename="$(find xarm_description)/urdf/xarm_device.urdf.xacro" /> -->
   <!-- Material Definition -->
   <material name="yellow">
@@ -26,5 +27,5 @@
       <mass value="10"/>
       <origin rpy="0 0 0" xyz="0 0 0"/>
-      <inertia ixx="0.008333333333" ixy="0" ixz="0" iyy="0.0.06041666667" iyz="0" izz="0.0.06041666667"/>
+      <inertia ixx="0.008333333333" ixy="0" ixz="0" iyy="0.06041666667" iyz="0" izz="0.06041666667"/>
     </inertial>
   </link>
@@ -47,5 +48,5 @@
       <mass value="0.5"/>
       <origin rpy="0 0 0" xyz="0 0 0"/>
-      <inertia ixx="0.0.06041666667" ixy="0" ixz="0" iyy="0.0008333333333" iyz="0" izz="0.0.06041666667"/>
+      <inertia ixx="0.06041666667" ixy="0" ixz="0" iyy="0.0008333333333" iyz="0" izz="0.06041666667"/>
     </inertial>
   </link>
@@ -67,5 +68,5 @@
       <mass value="0.5"/>
       <origin rpy="0 0 0" xyz="0 0 0"/>
-      <inertia ixx="0.0.06041666667" ixy="0" ixz="0" iyy="0.0.06041666667" iyz="0" izz="0.0008333333333"/>
+      <inertia ixx="0.06041666667" ixy="0" ixz="0" iyy="0.06041666667" iyz="0" izz="0.0008333333333"/>
     </inertial>
   </link>
@@ -113,5 +114,5 @@
   <!-- Joints  -->
   <joint name="world_to_base_link_joint" type="fixed">
-      <origin xyz="0.285 0 0.005" rpy="0 0 0"/>
+      <origin xyz="-0.5 -0.835 0.005" rpy="0 0 0"/>
       <parent link="world"/>
       <child link="base_link"/>
@@ -122,5 +123,5 @@
       <child link="x_link"/>
       <axis xyz="1 0 0"/>
-      <limit effort="50" velocity="0.01" lower="-0.6" upper="0.6"/>
+      <limit effort="50" velocity="0.01" lower="-0.5" upper="0.5"/>
       <dynamics damping="100.0" friction="100.0"/>
   </joint>

File: xarm6_control_trainig/urdf/tennis_robot_cylindrical.urdf.xacro (robot description, xacro)
@@ -1,4 +1,5 @@
 <?xml version="1.0"?>
 <robot xmlns:xacro="http://www.ros.org/wiki/xacro"  name="tennis_ball">
+  <!-- <xacro:include filename="$(find xarm_description)/urdf/xarm_device.urdf.xacro" /> -->
   <!-- Material Definition -->
   <material name="yellow">
@@ -29,10 +30,10 @@
     </inertial>
   </link>
-  <!-- The gantry robot -->
-  <link name="x_link">
+  <!-- The cylindrical robot -->
+  <link name="theta_link">
     <visual>
-      <origin xyz="0 0 0" rpy="0 0 0"/>
+      <origin xyz="0 0.380 0" rpy="0 0 0"/>
       <geometry>
-        <box size="0.01 1.2 0.01"/>
+        <box size="0.01 0.75 0.01"/>
       </geometry>
       <material name="black"/>
@@ -41,5 +42,5 @@
       <origin xyz="0 0 0" rpy="0 0 0"/>
       <geometry>
-        <box size="0.01 1.2 0.01"/>
+        <box size="0.01 0.75 0.01"/>
       </geometry>
     </collision>
@@ -50,9 +51,9 @@
     </inertial>
   </link>
-  <link name="y_link">
+  <link name="r_link">
     <visual>
       <origin xyz="0 0 0" rpy="0 0 0"/>
       <geometry>
-        <box size="0.01 0.01 1.2"/>
+        <box size="0.01 0.01 2.0"/>
       </geometry>
       <material name="black"/>
@@ -61,5 +62,5 @@
       <origin xyz="0 0 0" rpy="0 0 0"/>
       <geometry>
-        <box size="0.01 0.01 1.2"/>
+        <box size="0.01 0.01 2.0"/>
       </geometry>
     </collision>
@@ -81,5 +82,5 @@
       <origin xyz="0 0 0" rpy="0 0 0"/>
       <geometry>
-        <box size="0.01 0.01 0.1"/>
+        <box size="0.01 0.01 0.01"/>
       </geometry>
     </collision>
@@ -87,5 +88,5 @@
       <mass value="0.5"/>
       <origin rpy="0 0 0" xyz="0 0 0"/>
-      <inertia ixx="0.0008333333333" ixy="0" ixz="0" iyy="0.0008333333333" iyz="0" izz="0.0008333333333"/>
+      <inertia ixx="0.0.008333333333" ixy="0" ixz="0" iyy="0.0008333333333" iyz="0" izz="0.0.008333333333"/>
     </inertial>
   </link>
@@ -113,30 +114,30 @@
   <!-- Joints  -->
   <joint name="world_to_base_link_joint" type="fixed">
-      <origin xyz="0.285 0 0.005" rpy="0 0 0"/>
+      <origin xyz="-0.2 -0.415 0.005" rpy="0 0 0"/>
       <parent link="world"/>
       <child link="base_link"/>
   </joint>
-  <joint name="x_joint" type="prismatic">
-      <origin xyz="0 0.605 0" rpy="0 0 0"/>
+  <joint name="theta_joint" type="revolute">
+      <axis xyz="0 0 1"/>
+      <origin xyz="0 0 0" rpy="0 0 0"/>
       <parent link="base_link"/>
-      <child link="x_link"/>
-      <axis xyz="1 0 0"/>
-      <limit effort="50" velocity="0.01" lower="-0.6" upper="0.6"/>
+      <child link="theta_link"/>
+      <limit effort="50" velocity="0.01" lower="-1.5707" upper="1.5707"/>
       <dynamics damping="100.0" friction="100.0"/>
   </joint>
-  <joint name="y_joint" type="prismatic">
-      <origin xyz="0 0 0.605" rpy="0 0 0"/>
-      <parent link="x_link"/>
-      <child link="y_link"/>
+  <joint name="r_joint" type="prismatic">
+      <origin xyz="0 0.505 1.005" rpy="0 0 0"/>
+      <parent link="theta_link"/>
+      <child link="r_link"/>
       <axis xyz="0 1 0"/>
-      <limit effort="50" velocity="0.01" lower="-0.6" upper="0.6"/>
+      <limit effort="50" velocity="0.01" lower="-0.35" upper="0.1"/>
       <dynamics damping="100.0" friction="100.0"/>
   </joint>
   <joint name="z_joint" type="prismatic">
-      <origin xyz="0 -0.01 0" rpy="0 0 0"/>
-      <parent link="y_link"/>
+      <origin xyz="0 -0.005 0" rpy="0 0 0"/>
+      <parent link="r_link"/>
       <child link="z_link"/>
       <axis xyz="0 0 1"/>
-      <limit effort="50" velocity="0.01" lower="-0.1" upper="0.6"/>
+      <limit effort="50" velocity="0.01" lower="-0.2" upper="0.75"/>
       <dynamics damping="100.0" friction="100.0"/>
   </joint>
@@ -146,5 +147,5 @@
       <child link="ball"/>
   </joint>
-  <xacro:include filename="gazebo_plugin.xacro" />
+  <xacro:include filename="gazebo_plugin_cylindrical.xacro" />
 </robot>
-<!-- ros2 topic pub -1 /set_joint_trajectory trajectory_msgs/msg/JointTrajectory  '{header: {frame_id: world}, joint_names: [x_joint, y_joint, z_joint], points: [{positions: {0.3,0.3,0.3}, velocities: {0.02,0.01,0.01}}}]} -->
+<!-- ros2 topic pub -1 /set_joint_trajectory trajectory_msgs/msg/JointTrajectory  '{header: {frame_id: world}, joint_names: [theta_joint, r_joint, z_joint], points: [{positions: {1.0,0.3,0.3}]}' -->
