Commit message: update the URDF for new gzebo ignition

File: xarm6_control_trainig/urdf/tennis_robot_cylindrical_gz.urdf.xacro (robot description, xacro)
@@ -1,6 +1,22 @@
 <?xml version="1.0"?>
-<robot xmlns:xacro="http://www.ros.org/wiki/xacro"  name="tennis_ball">
-  <!-- <xacro:include filename="$(find xarm_description)/urdf/xarm_device.urdf.xacro" /> -->
-  <!-- Material Definition -->
+<!--
+  New-Gazebo (Ignition Fortress / gz-sim 6) description of the CYLINDRICAL
+  tennis-ball gantry target robot.  Parallel to the Classic
+  `tennis_robot_cylindrical.urdf.xacro` which is left untouched.
+  Link and joint names are IDENTICAL to the Classic cylindrical model
+  (theta_joint / r_joint / z_joint) so downstream scripts stay compatible.
+  Differences vs the Classic cylindrical file (all deliberate, noted here):
+    - Includes gazebo_plugin_cylindrical_gz.xacro (Ignition system plugins +
+      Fortress materials) instead of the Classic gazebo_plugin_cylindrical.xacro.
+    - Fixed several inertia values that were malformed doubles in the Classic
+      file (e.g. "0.0.06041666667", "0.0008333333333" written as
+      "0.0.008333333333").  Those strings are not valid numbers and would be
+      rejected by the URDF parser / SDF converter.  The intended magnitudes
+      were obvious from the matching well-formed values elsewhere, so they are
+      restored to 0.06041666667 / 0.008333333333 / 0.0008333333333 as
+      appropriate.  Masses, joint limits and damping are otherwise preserved.
+-->
+<robot xmlns:xacro="http://www.ros.org/wiki/xacro" name="tennis_ball">
+  <!-- Material Definition (URDF-side, used by robot_state_publisher / RViz) -->
   <material name="yellow">
     <color rgba="1 1 0 1"/>
@@ -22,5 +38,6 @@
       <mass value="10"/>
       <origin rpy="0 0 0" xyz="0 0 0"/>
-      <inertia ixx="0.008333333333" ixy="0" ixz="0" iyy="0.0.06041666667" iyz="0" izz="0.0.06041666667"/>
+      <!-- was iyy/izz "0.0.06041666667" (invalid) -> 0.06041666667 -->
+      <inertia ixx="0.008333333333" ixy="0" ixz="0" iyy="0.06041666667" iyz="0" izz="0.06041666667"/>
     </inertial>
   </link>
@@ -37,5 +54,6 @@
       <mass value="0.5"/>
       <origin rpy="0 0 0" xyz="0 0 0"/>
-      <inertia ixx="0.0.06041666667" ixy="0" ixz="0" iyy="0.0008333333333" iyz="0" izz="0.0.06041666667"/>
+      <!-- was ixx/izz "0.0.06041666667" (invalid) -> 0.06041666667 -->
+      <inertia ixx="0.06041666667" ixy="0" ixz="0" iyy="0.0008333333333" iyz="0" izz="0.06041666667"/>
     </inertial>
   </link>
@@ -51,5 +69,6 @@
       <mass value="0.5"/>
       <origin rpy="0 0 0" xyz="0 0 0"/>
-      <inertia ixx="0.0.06041666667" ixy="0" ixz="0" iyy="0.0.06041666667" iyz="0" izz="0.0008333333333"/>
+      <!-- was ixx/iyy "0.0.06041666667" (invalid) -> 0.06041666667 -->
+      <inertia ixx="0.06041666667" ixy="0" ixz="0" iyy="0.06041666667" iyz="0" izz="0.0008333333333"/>
     </inertial>
   </link>
@@ -65,5 +84,6 @@
       <mass value="0.5"/>
       <origin rpy="0 0 0" xyz="0 0 0"/>
-      <inertia ixx="0.0.008333333333" ixy="0" ixz="0" iyy="0.0008333333333" iyz="0" izz="0.0.008333333333"/>
+      <!-- was ixx/izz "0.0.008333333333" (invalid) -> 0.008333333333 -->
+      <inertia ixx="0.008333333333" ixy="0" ixz="0" iyy="0.0008333333333" iyz="0" izz="0.008333333333"/>
     </inertial>
   </link>
@@ -100,6 +120,6 @@
       <parent link="base_link"/>
       <child link="theta_link"/>
-      <limit effort="50" velocity="0.01" lower="-1.5707" upper="1.5707"/>
-      <dynamics damping="100.0" friction="100.0"/>
+      <limit effort="1000" velocity="5.0" lower="-1.5707" upper="1.5707"/>
+      <dynamics damping="1.0" friction="0.0"/>
   </joint>
   <joint name="r_joint" type="prismatic">
@@ -108,6 +128,6 @@
       <child link="r_link"/>
       <axis xyz="0 1 0"/>
-      <limit effort="50" velocity="0.01" lower="-0.35" upper="0.1"/>
-      <dynamics damping="100.0" friction="100.0"/>
+      <limit effort="1000" velocity="5.0" lower="-0.35" upper="0.1"/>
+      <dynamics damping="1.0" friction="0.0"/>
   </joint>
   <joint name="z_joint" type="prismatic">
@@ -116,6 +136,6 @@
       <child link="z_link"/>
       <axis xyz="0 0 1"/>
-      <limit effort="50" velocity="0.01" lower="-0.2" upper="0.75"/>
-      <dynamics damping="100.0" friction="100.0"/>
+      <limit effort="1000" velocity="5.0" lower="-0.2" upper="0.75"/>
+      <dynamics damping="1.0" friction="0.0"/>
   </joint>
   <joint name="fixed_joint" type="fixed">
@@ -124,5 +144,15 @@
       <child link="ball"/>
   </joint>
-  <xacro:include filename="gazebo_plugin_cylindrical.xacro" />
+  <!-- Ignition Fortress system plugins + Fortress materials -->
+  <xacro:include filename="gazebo_plugin_cylindrical_gz.xacro" />
 </robot>
-<!-- ros2 topic pub -1 /set_joint_trajectory trajectory_msgs/msg/JointTrajectory  '{header: {frame_id: world}, joint_names: [theta_joint, r_joint, z_joint], points: [{positions: {1.0,0.3,0.3}]}' -->
+<!--
+  How to move the ball (Fortress path):
+  The ros_gz_bridge maps ROS topic /set_joint_trajectory
+  (trajectory_msgs/msg/JointTrajectory) into the gz topic
+  /model/tennis_ball/set_joint_trajectory which the
+  JointTrajectoryController system consumes.  Example:
+  ros2 topic pub -1 /set_joint_trajectory trajectory_msgs/msg/JointTrajectory \
+    '{header: {frame_id: world}, joint_names: [theta_joint, r_joint, z_joint], \
+      points: [{positions: [0.5, -0.1, 0.3]}]}'
+-->

Commit message: adding moveit

File: xarm6_control_trainig/urdf/tennis_robot_cylindrical_gz.urdf.xacro (robot description, xacro)
@@ -18,4 +18,10 @@
 -->
 <robot xmlns:xacro="http://www.ros.org/wiki/xacro" name="tennis_ball">
+  <!-- show_frame: when true, the black gantry frame (base/theta/r/z links) is
+       rendered; when false (default) only the ball is visible. Collision and
+       inertia are always present regardless, so physics is unchanged.
+       Driven by the 'show_frame' launch argument. -->
+  <xacro:arg name="show_frame" default="false"/>
+  <xacro:property name="show_frame" value="$(arg show_frame)"/>
   <!-- Material Definition (URDF-side, used by robot_state_publisher / RViz) -->
   <material name="yellow">
@@ -29,5 +35,12 @@
   <link name="base_link">
     <origin xyz="0 0 0" rpy="0 0 0"/>
-    <!-- gantry frame visual hidden (physics kept via collision below) -->
+    <xacro:if value="${show_frame}">
+      <visual>
+        <geometry>
+          <box size="1.2 0.01 0.01"/>
+        </geometry>
+        <material name="black"/>
+      </visual>
+    </xacro:if>
     <collision>
       <geometry>
@@ -44,5 +57,13 @@
   <!-- The cylindrical robot -->
   <link name="theta_link">
-    <!-- gantry frame visual hidden (physics kept via collision below) -->
+    <xacro:if value="${show_frame}">
+      <visual>
+        <origin xyz="0 0.380 0" rpy="0 0 0"/>
+        <geometry>
+          <box size="0.01 0.75 0.01"/>
+        </geometry>
+        <material name="black"/>
+      </visual>
+    </xacro:if>
     <collision>
       <origin xyz="0 0 0" rpy="0 0 0"/>
@@ -59,5 +80,13 @@
   </link>
   <link name="r_link">
-    <!-- gantry frame visual hidden (physics kept via collision below) -->
+    <xacro:if value="${show_frame}">
+      <visual>
+        <origin xyz="0 0 0" rpy="0 0 0"/>
+        <geometry>
+          <box size="0.01 0.01 2.0"/>
+        </geometry>
+        <material name="black"/>
+      </visual>
+    </xacro:if>
     <collision>
       <origin xyz="0 0 0" rpy="0 0 0"/>
@@ -74,5 +103,13 @@
   </link>
   <link name="z_link">
-    <!-- gantry frame visual hidden (physics kept via collision below) -->
+    <xacro:if value="${show_frame}">
+      <visual>
+        <origin xyz="0 0 0" rpy="0 0 0"/>
+        <geometry>
+          <box size="0.01 0.01 0.01"/>
+        </geometry>
+        <material name="black"/>
+      </visual>
+    </xacro:if>
     <collision>
       <origin xyz="0 0 0" rpy="0 0 0"/>
